File: 10-gbe-expansion.kicad_pcb (KiCad board)
At the start: 2 copper layers, 0 parts

Commit message: [#80813] Draft X710 power, PCIe and 10GbE interfaces
Parts:
- added U1: EZX710AT2_S_LMR5, antmicro-footprints:FCBGA-503_22x22mm_Layout21x24_P1mm, F.Cu at (102.5, 68.3)
Other:
- board outline added: 80.5 x 76.5 mm
- board text added: "PCB SHA ########"
