File: ideal-diode.kicad_sch (KiCad schematic)
At the start: 4 parts, among them Q1 SQS401EN-T1_BE3, U11 LTC4412IS6

Commit message: [#85196] Re-annotate schematic
Parts:
- renumbered C167 to C200, C168 to C201, Q1 to Q2
Changed lines of the file:
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@@
 		(on_board yes)
 		(dnp no)
-		(property "Reference" "C168"
+		(property "Reference" "C201"
 			(at 228.346 153.67 90)
 			(effects
@@
 			(project "10-gbe-expansion"
 				(path "/04bda987-e5eb-48b4-9e90-d8211dc11b39/3d913a88-b6f3-4148-9b3d-882d5df37282/151969d2-a4e0-4623-bed4-6527ef713b4c"
-					(reference "C170")
+					(reference "C203")
 					(unit 1)
 				)
 				(path "/04bda987-e5eb-48b4-9e90-d8211dc11b39/3d913a88-b6f3-4148-9b3d-882d5df37282/6ef59793-527b-4d85-9643-0ce8a14d0e9d"
-					(reference "C168")
+					(reference "C201")
 					(unit 1)
 				)
@@
 		(on_board yes)
 		(dnp no)
-		(property "Reference" "C167"
+		(property "Reference" "C200"
 			(at 189.738 153.67 90)
 			(effects
@@
 			(project "10-gbe-expansion"
 				(path "/04bda987-e5eb-48b4-9e90-d8211dc11b39/3d913a88-b6f3-4148-9b3d-882d5df37282/151969d2-a4e0-4623-bed4-6527ef713b4c"
-					(reference "C169")
+					(reference "C202")
 					(unit 1)
 				)
 				(path "/04bda987-e5eb-48b4-9e90-d8211dc11b39/3d913a88-b6f3-4148-9b3d-882d5df37282/6ef59793-527b-4d85-9643-0ce8a14d0e9d"
-					(reference "C167")
+					(reference "C200")
 					(unit 1)
 				)
@@
 		(dnp no)
 		(fields_autoplaced yes)
-		(property "Reference" "#PWR0290"
+		(property "Reference" "#PWR0328"
 			(at 196.85 168.91 0)
 			(effects
@@
 			(project "10-gbe-expansion"
 				(path "/04bda987-e5eb-48b4-9e90-d8211dc11b39/3d913a88-b6f3-4148-9b3d-882d5df37282/151969d2-a4e0-4623-bed4-6527ef713b4c"
-					(reference "#PWR0292")
+					(reference "#PWR0330")
 					(unit 1)
 				)
 				(path "/04bda987-e5eb-48b4-9e90-d8211dc11b39/3d913a88-b6f3-4148-9b3d-882d5df37282/6ef59793-527b-4d85-9643-0ce8a14d0e9d"
-					(reference "#PWR0290")
+					(reference "#PWR0328")
 					(unit 1)
 				)
@@
 		(dnp no)
 		(fields_autoplaced yes)
-		(property "Reference" "#PWR0291"
+		(property "Reference" "#PWR0329"
 			(at 226.06 168.91 0)
 			(effects
@@
 			(project "10-gbe-expansion"
 				(path "/04bda987-e5eb-48b4-9e90-d8211dc11b39/3d913a88-b6f3-4148-9b3d-882d5df37282/151969d2-a4e0-4623-bed4-6527ef713b4c"
-					(reference "#PWR0293")
+					(reference "#PWR0331")
 					(unit 1)
 				)
 				(path "/04bda987-e5eb-48b4-9e90-d8211dc11b39/3d913a88-b6f3-4148-9b3d-882d5df37282/6ef59793-527b-4d85-9643-0ce8a14d0e9d"
-					(reference "#PWR0291")
+					(reference "#PWR0329")
 					(unit 1)
 				)
@@
 		(on_board yes)
 		(dnp no)
-		(property "Reference" "Q1"
+		(property "Reference" "Q2"
 			(at 217.17 130.81 90)
 			(effects
@@
 			(project "10-gbe-expansion"
 				(path "/04bda987-e5eb-48b4-9e90-d8211dc11b39/3d913a88-b6f3-4148-9b3d-882d5df37282/151969d2-a4e0-4623-bed4-6527ef713b4c"
+					(reference "Q3")
+					(unit 1)
+				)
+				(path "/04bda987-e5eb-48b4-9e90-d8211dc11b39/3d913a88-b6f3-4148-9b3d-882d5df37282/6ef59793-527b-4d85-9643-0ce8a14d0e9d"
 					(reference "Q2")
 					(unit 1)
 				)
-				(path "/04bda987-e5eb-48b4-9e90-d8211dc11b39/3d913a88-b6f3-4148-9b3d-882d5df37282/6ef59793-527b-4d85-9643-0ce8a14d0e9d"
-					(reference "Q1")
-					(unit 1)
-				)
